Commit message: Add robot models
Add monocular, stereo and RGBD robot models.

File: urdf/rgbd_robot.urdf (robot description, URDF)
Before this commit: robot simple_robot, 9 links, 8 joints
Links:
- removed link camera
- added link stereo_camera_link, mass 0.001; collision box size=0.1 .02 .02; visual box size=0.1 0.02 0.02
Joints:
- removed joint camera_joint
- added joint robot_footprint_to_stereo_camera_joint: type fixed, parent chassis, child stereo_camera_link, origin xyz=0.15 0 0.15 rpy=0 0 0, axis 0 0 0
- joint hokuyo_joint: origin xyz=0.15 0 0.1 rpy=0 0 0 -> xyz=0.15 0 0.07 rpy=0 0 0
- joint imu_joint: origin xyz=0.15 0 0.05 rpy=0 0 0 -> xyz=0.15 0 0.12 rpy=0 0 0

File: urdf/stereo_robot.urdf (robot description, URDF)
Before this commit: robot simple_robot, 9 links, 8 joints
Links:
- removed link camera
- added link stereo_camera_link, mass 0.001; collision box size=0.1 .02 .02; visual box size=0.1 0.02 0.02
Joints:
- removed joint camera_joint
- added joint robot_footprint_to_stereo_camera_joint: type fixed, parent chassis, child stereo_camera_link, origin xyz=0.15 0 0.15 rpy=0 0 0, axis 0 0 0
- joint hokuyo_joint: origin xyz=0.15 0 0.1 rpy=0 0 0 -> xyz=0.15 0 0.07 rpy=0 0 0
- joint imu_joint: origin xyz=0.15 0 0.05 rpy=0 0 0 -> xyz=0.15 0 0.12 rpy=0 0 0
